File: project/ECAD/PCB-MachineThatDraws/PCB-MachineThatDraws.kicad_pcb (KiCad board)
At the start: 2 copper layers, 24 x 16 mm, 8 parts, among them J1 SD_Card_Device, J10 Conn_02x03_Odd_Even, J11 Conn_02x03_Odd_Even, J3 Switch, J4 Switch, U2 R-78E5.0-1.0

Commit message: Update PCB-MachineThatDraws.kicad_pcb
Parts:
- added C1: 100µF, makerspace-unilasalle:C_1206, F.Cu at (139.3, 40.8)
- added C3: C_Polarized_Small, Capacitor_SMD:CP_Elec_6.3x5.4, F.Cu at (129.5, 69.0)
- added C4: C_Polarized_Small, Capacitor_SMD:CP_Elec_6.3x5.4, F.Cu at (129.5, 77.1)
- added C5: 10µF, makerspace-unilasalle:C_1206, F.Cu at (139.3, 44.1)
- added C6: 10µF, makerspace-unilasalle:C_1206, F.Cu at (139.3, 47.5)
- added C7: 10uF, makerspace-unilasalle:C_1206, F.Cu at (139.3, 50.8)
- added C8: 100nF, makerspace-unilasalle:C_1206, F.Cu at (139.3, 54.2)
- added D1: Green, LED_SMD:LED_1206_3216Metric, F.Cu at (137.7, 87.6)
- added F1: Fuse, Fuse:Fuseholder_Blade_Mini_Keystone_3568, F.Cu at (25.2, 94.8)
- added J2: SDA/SCL/VCC/GND, Connector:NS-Tech_Grove_1x04_P2mm_Vertical, F.Cu at (59.0, 92.1)
- added J5: Moteur, Connector:NS-Tech_Grove_1x04_P2mm_Vertical, F.Cu at (66.5, 92.1)
- added J6: Moteur, Connector:NS-Tech_Grove_1x04_P2mm_Vertical, F.Cu at (74.0, 92.1)
- added J7: Barrel_Jack_Switch, Connector_BarrelJack:BarrelJack_GCT_DCJ200-10-A_Horizontal, F.Cu at (129.7, 41.1)
- added J8: Screw_Terminal_01x02, TerminalBlock:TerminalBlock_bornier-2_P5.08mm, F.Cu at (127.4, 60.4)
- added J9: Servo, Connector:FanPinHeader_1x03_P2.54mm_Vertical, F.Cu at (137.1, 81.6)
- added R1: 4.7K, makerspace-unilasalle:R_1206, F.Cu at (83.8, 72.2)
- added R2: 4.7K, makerspace-unilasalle:R_1206, F.Cu at (83.8, 75.5)
- added R3: 1K, makerspace-unilasalle:R_1206, F.Cu at (83.8, 78.8)
- added R4: 10k, makerspace-unilasalle:R_1206, F.Cu at (83.8, 82.1)
- added R5: 10k, makerspace-unilasalle:R_1206, F.Cu at (83.8, 85.4)
- added U1: ESP32-S3-UNO, makerspace-unilasalle:ESP_S3_UNO, B.Cu at (114.2, 36.2)
- J4: value Switch -> Limit_Switch_X
- moved J10 117.9 mm to (41.3, 94.7)
- moved J11 117.9 mm to (48.5, 94.7)
- moved A1 109.5 mm to (23.5, 72.5)
- moved A2 109.5 mm to (40.3, 72.5)
- moved U2 81.3 mm to (81.8, 95.8)
- moved J1 80.4 mm to (68.0, 87.5)
- moved J3 31.4 mm to (137.8, 67.6)
- moved J4 31.4 mm to (137.8, 74.2)
Connections:
- J1 pad 2: unconnected-(J1-CMD-Pad2) -> D11
- J1 pad 7: unconnected-(J1-DAT0-Pad7) -> D19
- J1 pad 8: D19 -> unconnected-(J1-DAT1-Pad8)
- J1 pad 9: D11 -> unconnected-(J1-DAT2-Pad9)

Commit message: Update PCB-MachineThatDraws.kicad_pcb
Parts:
- moved F1 163.8 mm to (189.0, 99.7), turned to 180 degrees
- moved J10 145.7 mm to (186.4, 81.7), turned to 90 degrees
- moved A1 142.0 mm to (165.0, 60.3), turned to 90 degrees
- moved J1 140.1 mm to (208.0, 85.5), turned to 180 degrees
- moved J11 139.4 mm to (186.4, 74.5), turned to 90 degrees
- moved J2 128.3 mm to (184.5, 65.5), turned to 90 degrees
- moved J6 126.8 mm to (196.5, 59.0), turned to 180 degrees
- moved J5 126.7 mm to (188.5, 58.0), turned to 180 degrees
- moved A2 125.5 mm to (165.0, 86.3), turned to 90 degrees
- moved R5 113.6 mm to (196.5, 71.4), turned to 180 degrees
- moved R4 113.0 mm to (196.5, 74.7), turned to 180 degrees
- moved R2 112.9 mm to (196.5, 81.3), turned to 180 degrees
- moved R3 112.7 mm to (196.5, 78.0), turned to 180 degrees
- moved R1 98.7 mm to (181.0, 89.5)
- moved U2 98.2 mm to (174.9, 64.8), turned to 180 degrees
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Other:
- outline, holes or cut-outs redrawn

Commit message: Update PCB-MachineThatDraws.kicad_pcb
Routing:
- net GND: track 0.00 -> 9.75 mm
Changed lines of the file:
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@@
 		)
+	)
+	(segment
+		(start 211.7723 100.4172)
+		(end 207.8295 100.4172)
+		(width 0.2)
+		(layer "B.Cu")
+		(net 13)
+	)
+	(segment
+		(start 206.15 98.7377)
+		(end 206.15 98.3)
+		(width 0.2)
+		(layer "B.Cu")
+		(net 13)
+	)
+	(segment
+		(start 213.65 98.2)
+		(end 213.65 98.5395)
+		(width 0.2)
+		(layer "B.Cu")
+		(net 13)
+	)
+	(segment
+		(start 213.65 98.5395)
+		(end 211.7723 100.4172)
+		(width 0.2)
+		(layer "B.Cu")
+		(net 13)
+	)
+	(segment
+		(start 207.8295 100.4172)
+		(end 206.15 98.7377)
+		(width 0.2)
+		(layer "B.Cu")
+		(net 13)
 	)
 	(zone

Commit message: PCB up
Parts:
- J1: footprint Connector_Card:SD_Card_Device_16mm_SlotDepth -> makerspace-unilasalle:SD_Hirose_DM1AA_SF_PEJ82
- J10, J11: moved to B.Cu
- U1: moved to F.Cu
- moved J3 111.3 mm to (102.5, 77.5)
- moved C3 101.8 mm to (103.5, 68.8), turned to 90 degrees
- moved J7 94.8 mm to (110.8, 40.0), turned to -90 degrees
- moved J4 92.7 mm to (121.0, 75.3)
- moved J8 92.4 mm to (115.4, 39.5)
- moved J1 91.6 mm to (117.5, 99.5), turned to 0 degrees
- moved F1 86.2 mm to (128.7, 38.0), turned to -90 degrees
- moved R5 85.6 mm to (111.5, 81.3), turned to 0 degrees
- moved J5 84.9 mm to (103.7, 54.8), turned to 0 degrees
- moved C1 82.3 mm to (142.5, 90.0)
- moved C5 80.5 mm to (134.4, 46.3)
- moved U1 79.2 mm to (99.0, 62.6), turned to 90 degrees
- moved C7 78.3 mm to (139.5, 82.5), turned to 180 degrees
- moved R4 77.3 mm to (119.5, 81.3)
- moved C6 76.0 mm to (139.4, 46.3), turned to 180 degrees
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Connections:
- U1 pad 1: (no net) -> unconnected-(U1-GPIO0-Pad1)
- U1 pad 10: (no net) -> D8
- U1 pad 11: (no net) -> D07
- U1 pad 12: (no net) -> D19
- U1 pad 13: (no net) -> D05
- U1 pad 14: (no net) -> unconnected-(U1-GPIO4/ADC1_CH3-Pad14)
- U1 pad 15: (no net) -> unconnected-(U1-GPIO44/U0RXD-Pad15)
- U1 pad 16: (no net) -> unconnected-(U1-GPIO43/U0TXD-Pad16)
- U1 pad 17: (no net) -> D18
- U1 pad 18: (no net) -> D10
- U1 pad 19: (no net) -> unconnected-(U1-GPIO19/USB_D--Pad19)
- U1 pad 2: (no net) -> unconnected-(U1-5V-Pad2)
- U1 pad 20: (no net) -> unconnected-(U1-GPIO20/USB_D+-Pad20)
- U1 pad 21: (no net) -> D14
- U1 pad 22: (no net) -> unconnected-(U1-GPIO14/ADC2_CH3-Pad22)
- U1 pad 23: (no net) -> unconnected-(U1-GPIO21-Pad23)
- U1 pad 24: (no net) -> Enable
- U1 pad 25: (no net) -> unconnected-(U1-GPIO10/ADC1_CH9-Pad25)
- U1 pad 26: (no net) -> D11
- U1 pad 27: (no net) -> D13
- U1 pad 28: (no net) -> D12
- U1 pad 29: (no net) -> GND
- U1 pad 3: (no net) -> unconnected-(U1-RST-Pad3)
- U1 pad 30: (no net) -> unconnected-(U1-RST-Pad30)
- U1 pad 31: (no net) -> SDA 
- U1 pad 32: (no net) -> SCL
- U1 pad 4: (no net) -> +3.3V
- U1 pad 6: (no net) -> GND
- U1 pad 7: (no net) -> GND
- U1 pad 8: (no net) -> +5V
- U1 pad 9: (no net) -> D9
Routing:
- net GND: track 9.75 -> 87.4 mm
- net +3.3V: track 0.00 -> 63.9 mm
- net +12V: track 0.00 -> 23.6 mm
- net Net-(A2-MS1): track 0.00 -> 22.4 mm
- net Net-(A2-MS2): track 0.00 -> 18.9 mm
- net Net-(A2-MS3): track 0.00 -> 15.2 mm
- net Net-(A1-MS3): track 0.00 -> 14.8 mm
- net +5V: track 0.00 -> 11.4 mm
- net Net-(A1-MS2): track 0.00 -> 11.2 mm
- net Net-(J8-Pin_1): track 0.00 -> 9.65 mm
- net Net-(J8-Pin_2): track 0.00 -> 8.80 mm
- net SDA: track 0.00 -> 8.45 mm
- net Net-(A1-MS1): track 0.00 -> 7.62 mm
- net Net-(A1-2B): track 0.00 -> 7.59 mm
- net Net-(A1-2A): track 0.00 -> 7.36 mm
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Other:
- board size 24 x 16 mm -> 52.5 x 65 mm

Commit message: 10-04
Other:
- board size 52.5 x 65 mm -> 52.5 x 83 mm
Changed lines of the file:
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@@
 	(gr_line
 		(start 149 34.5)
-		(end 149 99.5)
+		(end 149 117.5)
 		(stroke
 			(width 0.05)
@@
 	)
 	(gr_line
-		(start 135 99.5)
-		(end 100.5 99.5)
+		(start 149 117.5)
+		(end 96.5 117.5)
 		(stroke
 			(width 0.05)
@@
 	)
 	(gr_line
-		(start 96.5 99.5)
+		(start 96.5 117.5)
 		(end 96.5 34.5)
-		(stroke
-			(width 0.05)
-			(type default)
-		)
-		(layer "Edge.Cuts")
-	)
-	(gr_line
-		(start 149 99.5)
-		(end 135 99.5)
-		(stroke
-			(width 0.05)
-			(type default)
-		)
-		(layer "Edge.Cuts")
-	)
-	(gr_line
-		(start 100.5 99.5)
-		(end 96.5 99.5)
 		(stroke
 			(width 0.05)
@@
 		(polygon
 			(pts
-				(xy 96.5 34.5) (xy 149 34.5) (xy 149 99.5) (xy 135 99.5) (xy 133.5 99.5) (xy 102 99.5) (xy 100.5 99.5)
-				(xy 96.5 99.5)
+				(xy 149 34.5) (xy 96.5 34.5) (xy 96.5 117.5) (xy 149 117.5)
 			)
 		)

Commit message: pcb update
Routing:
- net GND: track 87.4 -> 279.2 mm, vias 0 -> 2
- net +5V: track 11.4 -> 92.7 mm, vias 0 -> 6
- net +3.3V: track 63.9 -> 144.5 mm, vias 0 -> 1
- net Enable: track 0.00 -> 63.4 mm, vias 0 -> 1
- net +12V: track 23.6 -> 83.8 mm
- net D11: track 0.00 -> 60.1 mm
- net D12: track 0.00 -> 57.8 mm, vias 0 -> 2
- net D07: track 0.00 -> 56.9 mm, vias 0 -> 2
- net D13: track 0.00 -> 47.7 mm, vias 0 -> 2
- net D10: track 0.00 -> 46.6 mm, vias 0 -> 2
- net D9: track 0.00 -> 42.6 mm, vias 0 -> 1
- net D05: track 4.33 -> 43.8 mm, vias 0 -> 1
- net D18: track 0.00 -> 38.7 mm, vias 0 -> 1
- net D14: track 0.00 -> 29.9 mm, vias 0 -> 1
- net D19: track 3.82 -> 21.3 mm
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
Commit message: Add files via upload
Routing:
- net GND: track 279.2 -> 298.7 mm, vias 2 -> 1
- net +5V: track 92.7 -> 105.0 mm, vias 6 -> 0
- net D10: track 46.6 -> 57.0 mm, vias 2 -> 1
- net D11: track 60.1 -> 69.7 mm
- net D13: track 47.7 -> 39.9 mm, vias 2 -> 0
- net Enable: track 63.4 -> 56.3 mm
- net D12: track 57.8 -> 61.8 mm, vias 2 -> 0
- net D07: track 56.9 -> 54.1 mm, vias 2 -> 1
- net +3.3V: track 144.5 -> 144.2 mm, vias 1 -> 0
Other:
- board size 52.5 x 83 mm -> 53.5 x 83 mm
